File: Cyberdeck_TD_Carrier/Cyberdeck_TD_Carrier.kicad_pcb (KiCad board)
At the start: 4 copper layers, 180 x 80 mm, 205 parts, among them J78 HDMI_A, J79 USB3_A_Stacked, J80 USB_A_Stacked, J81 RJ45_RB1-125B8G1A, J82 Bus_M.2_Socket_M, J83 Bus_M.2_Socket_E, J84 USB_C_Receptacle_USB2.0, J85 BAT_TERM, M78 Fan_4pin, Q78 2N7002, Q79 2SK3018, Q80 2SK3018, Q81 2SK3018, Q82 FDMC8327L, Q83 FDMC8327L, Q84 2N7002, SW78 PWR_BTN, U78 TPAZ1023-04F, U79 TPAZ1023-04F, U80 ULC0524P, U81 ULC0524P, U82 ULC0524P, U83 RTL8111H-CG-RH, U84 ULC0524P, U85 ULC0524P, U86 LTC4162-L42, U87 CH224K, U88 SY8253ADC, U89 SY8253ADC, U90 MAX98365AEWC+, Y78 25MHz

Commit message: Add files via upload
Parts:
- added LS78: Speaker, Connector_PinHeader_2.00mm:PinHeader_1x02_P2.00mm_Vertical, F.Cu at (238.4, 105.2)
- moved C156 7.73 mm to (230.0, 104.5)
- moved C155 6.96 mm to (231.0, 101.7), turned to -90 degrees
- moved C111 6.44 mm to (102.6, 124.0), turned to 90 degrees
- moved C110 6.42 mm to (101.6, 124.0), turned to 90 degrees
- moved C116 6.33 mm to (103.6, 124.0), turned to 90 degrees
- moved C117 6.33 mm to (104.5, 124.0), turned to 90 degrees
- moved C154 4.75 mm to (232.5, 101.7), turned to -90 degrees
- moved C153 3.68 mm to (234.0, 101.7), turned to -90 degrees
- moved D93 2.67 mm to (130.0, 130.4)
- moved R127 2.67 mm to (127.4, 131.3)
- moved R81 2.67 mm to (127.4, 129.9)
- moved R83 2.58 mm to (121.4, 114.8), turned to 90 degrees
- moved R80 2.53 mm to (219.7, 110.8)
- moved R82 1.55 mm to (123.2, 115.8)
- moved R78 1.38 mm to (145.4, 124.4)
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Connections:
- A78 pad 162: unconnected-(A78-I2S_SCLK-Pad162) -> BCLK
- A78 pad 164: unconnected-(A78-I2S_SFRM-Pad164) -> FCLK
- A78 pad 166: unconnected-(A78-I2S_TXD-Pad166) -> AUDIO
Routing:
- net /~{PWR_LED}/~{PSON}: track 84.2 -> 246.7 mm, vias 2 -> 4
- net /LattePanda Module/SLS_S3: track 45.7 -> 203.6 mm, vias 1 -> 3
- net /LattePanda Module/REFCLK0-: track 0.00 -> 149.2 mm
- net /LattePanda Module/REFCLK0+: track 0.00 -> 149.1 mm
- net /~{PLT_RST}: track 29.8 -> 167.0 mm, vias 2 -> 3
- net /LattePanda Module/SUSCLK_WIFI: track 0.00 -> 124.5 mm, vias 0 -> 9
- net +BATT: track 0.00 -> 112.9 mm, vias 0 -> 2
- net /M.2 E&M Key/CON_PCIE_TX_1+: track 0.00 -> 109.4 mm
- net /M.2 E&M Key/CON_PCIE_TX_1-: track 0.00 -> 109.3 mm
- net /HDMI/DDI_B_DDC_SDA: track 3.39 -> 110.5 mm, vias 0 -> 2
- net /HDMI/DDI_B_DDC_SCL: track 3.32 -> 105.0 mm, vias 0 -> 6
- net /HDMI/DDI_B_HPD: track 3.51 -> 102.9 mm, vias 0 -> 6
- net /HDMI/DDI_B_TX1-: track 0.00 -> 91.2 mm, vias 0 -> 2
- net /HDMI/DDI_B_TX0-: track 0.00 -> 91.2 mm, vias 0 -> 2
- net /HDMI/DDI_B_TX1+: track 0.00 -> 91.1 mm, vias 0 -> 2
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