File: Cyberdeck_TD_Carrier/LattePanda Module.kicad_sch (KiCad schematic)
At the start: 16 parts, among them U90 MAX98365AEWC+

Commit message: Add files via upload
Parts:
- LS78: footprint (none) -> Connector_PinHeader_2.00mm:PinHeader_1x02_P2.00mm_Vertical
Connections:
- net AUDIO: now also A78.166 (I2S_TXD)
- net BCLK: now also A78.162 (I2S_SCLK)
- net FCLK: now also A78.164 (I2S_SFRM)
- no-connect marks 91 -> 88
Changed lines of the file:
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@@
 	)
 	(no_connect
-		(at 351.79 264.16)
-	)
-	(no_connect
 		(at 270.51 190.5)
 	)
@@
 	)
 	(no_connect
-		(at 351.79 269.24)
-	)
-	(no_connect
 		(at 270.51 203.2)
 	)
@@
 	)
 	(no_connect
-		(at 351.79 266.7)
-	)
-	(no_connect
 		(at 351.79 283.21)
 	)
@@
 	(wire
 		(pts
+			(xy 351.79 266.7) (xy 356.87 266.7)
+		)
+		(stroke
+			(width 0)
+			(type default)
+		)
+	)
+	(wire
+		(pts
 			(xy 351.79 226.06) (xy 368.3 226.06)
 		)
@@
 	(wire
 		(pts
+			(xy 351.79 269.24) (xy 356.87 269.24)
+		)
+		(stroke
+			(width 0)
+			(type default)
+		)
+	)
+	(wire
+		(pts
 			(xy 309.88 44.45) (xy 309.88 55.88)
 		)
@@
 	(wire
 		(pts
+			(xy 351.79 264.16) (xy 356.87 264.16)
+		)
+		(stroke
+			(width 0)
+			(type default)
+		)
+	)
+	(wire
+		(pts
 			(xy 238.76 233.68) (xy 270.51 233.68)
 		)
@@
 		)
 	)
-	(global_label "3V3"
+	(global_label "FCLK"
 		(shape input)
-		(at 415.29 332.74 180)
+		(at 356.87 266.7 0)
 		(fields_autoplaced yes)
 		(effects
@@
 				(size 1.27 1.27)
 			)
-			(justify right)
+			(justify left)
 		)
 		(property "Intersheetrefs" "${INTERSHEET_REFS}"
-			(at 408.7972 332.74 0)
+			(at 364.5119 266.7 0)
 			(effects
 				(font
 					(size 1.27 1.27)
 				)
-				(justify right)
+				(justify left)
+				(hide yes)
+			)
+		)
+	)
+	(global_label "AUDIO"
+		(shape input)
+		(at 356.87 269.24 0)
+		(fields_autoplaced yes)
+		(effects
+			(font
+				(size 1.27 1.27)
+			)
+			(justify left)
+		)
+		(property "Intersheetrefs" "${INTERSHEET_REFS}"
+			(at 365.4796 269.24 0)
+			(effects
+				(font
+					(size 1.27 1.27)
+				)
+				(justify left)
 				(hide yes)
 			)
@@
 		)
 	)
+	(global_label "BCLK"
+		(shape input)
+		(at 356.87 264.16 0)
+		(fields_autoplaced yes)
+		(effects
+			(font
+				(size 1.27 1.27)
+			)
+			(justify left)
+		)
+		(property "Intersheetrefs" "${INTERSHEET_REFS}"
+			(at 364.6933 264.16 0)
+			(effects
+				(font
+					(size 1.27 1.27)
+				)
+				(justify left)
+				(hide yes)
+			)
+		)
+	)
 	(global_label "AUDIO"
 		(shape input)
@@
 	)
 	(symbol
+		(lib_id "power:VDC")
+		(at 415.29 332.74 90)
+		(unit 1)
+		(exclude_from_sim no)
+		(in_bom yes)
+		(on_board yes)
+		(dnp no)
+		(fields_autoplaced yes)
+		(property "Reference" "#PWR0186"
+			(at 417.83 332.74 0)
+			(effects
+				(font
+					(size 1.27 1.27)
+				)
+				(hide yes)
+			)
+		)
+		(property "Value" "3V3"
+			(at 411.48 332.7399 90)
+			(effects
+				(font
+					(size 1.27 1.27)
+				)
+				(justify left)
+			)
+		)
+		(property "Footprint" ""
+			(at 415.29 332.74 0)
+			(effects
+				(font
+					(size 1.27 1.27)
+				)
+				(hide yes)
+			)
+		)
+		(property "Datasheet" ""
+			(at 415.29 332.74 0)
+			(effects
+				(font
+					(size 1.27 1.27)
+				)
+				(hide yes)
+			)
+		)
+		(property "Description" ""
+			(at 415.29 332.74 0)
+			(effects
+				(font
+					(size 1.27 1.27)
+				)
+				(hide yes)
+			)
+		)
+		(pin "1"
+		)
+		(instances
+			(project "Cyberdeck_TD_Carrier"
+				(path "/2a6d114a-7fd7-4207-b5f7-4ea9c34f36aa/6eee02c2-78c9-4e83-9ccf-e0f7690b57bf"
+					(reference "#PWR0186")
+					(unit 1)
+				)
+			)
+		)
+	)
+	(symbol
 		(lib_id "Device:C")
 		(at 406.4 341.63 180)
@@
 			)
 		)
-		(property "Footprint" ""
+		(property "Footprint" "Connector_PinHeader_2.00mm:PinHeader_1x02_P2.00mm_Vertical"
 			(at 410.21 314.96 0)
 			(effects
